File: hardware/stm32/bluepill.kicad_pcb (KiCad board)
At the start: 2 copper layers, 50 x 100 mm, 82 parts, among them J1 LCD, J10 S3, J11 S4, J12 S5, J13 S6, J14 RTC, J15 +5V, J16 Conn_01x02_Male, J17 ESP-01, J18 USART1, J19 Buttons, J2 SD Card, J3 Radio, J4 Outer, J5 Inner, J6 LED Power, J7 Open, J8 S1, J9 S2, Q1 IRLML2502, Q2 IRLML2502, Q3 IRLML2502, Q4 IRLML2502, Q5 IRLML2502, Q6 IRLML2502, U1 PC817, U10 PC817, U11 PC817, U12 LM1117-3.3, U2 24LC512, U3 bluepill, U4 PC817, U5 PC817, U6 PC817, U7 PC817, U8 PC817, U9 PC817

Commit message: KiCad 7.0
Other:
- net class 12V removed
- net class 3.3V removed
- net class 5V removed
- net class Default removed
- net class GND removed
- net class Strong removed
